File: PCB-Set-In-Stone-KiCAD/Set_In_Stone.kicad_pcb (KiCad board)
At the start: 2 copper layers, 144 x 114 mm, 9 parts, among them J1 TFT ILI9341 Cap Touch, J2 Joystick, J3 Conn_01x06, SW1 Blue Button, SW2 Green Button, SW3 Yellow Button, SW4 Red_Button, U1 ESP32-DEVKITC-32D

Commit message: Made finishing touches to PCB
In this update, I made the final touches for the PCB of the Set In Stone project.
Parts:
- added REF**: MountingHole_3.2mm_M3, MountingHole:MountingHole_3.2mm_M3, F.Cu at (215.0, 43.0)
- added REF**: MountingHole_3.2mm_M3, MountingHole:MountingHole_3.2mm_M3, F.Cu at (79.5, 43.5)
- added REF**: MountingHole_3.2mm_M3, MountingHole:MountingHole_3.2mm_M3, F.Cu at (215.5, 149.5)
- added REF**: MountingHole_3.2mm_M3, MountingHole:MountingHole_3.2mm_M3, F.Cu at (79.5, 149.5)
- moved J2 38.5 mm to (212.0, 123.0)
- moved J1 12.5 mm to (109.0, 66.5)
Routing:
- net SW: track 83.3 -> 120.6 mm
- net TFT_SCK: track 147.9 -> 110.8 mm
- net TFT_MOSI: track 232.8 -> 198.4 mm
- net VRX: track 66.2 -> 49.0 mm
- net VRY: track 65.6 -> 48.6 mm
- net +3V3: track 328.7 -> 345.6 mm
- net SD_CS: track 207.2 -> 193.6 mm
- net TFT SCL: track 80.4 -> 93.5 mm
- net TFT_LED: track 87.7 -> 100.7 mm
- net TFT_CS: track 71.8 -> 84.8 mm
- net TFT SDA: track 71.7 -> 84.7 mm
- net TFT_RST: track 129.2 -> 141.5 mm
- net TFT_DC: track 84.3 -> 94.2 mm
- net TFT MISO: track 122.1 -> 127.3 mm

Commit message: Made Wires Bigger and Made PCBWAY GERBER FILES
In this update, I redid the routing for the wires slightly so that there isnt redudant wires hopefully as well as increase the wire thickness for the general wiring as well as for the VCC which is the 3.3V in the diagram.
Parts:
- moved REF** 50.0 mm to (165.0, 43.5)
- moved U1 0.30 mm to (204.0, 74.3)
Routing:
- net TFT_MOSI: track 198.4 -> 385.8 mm
- net +3V3: track 345.6 -> 199.2 mm
- net GND: track 0.00 -> 72.2 mm, vias 0 -> 2
- net SW: track 120.6 -> 71.9 mm
- net SD_CS: track 193.6 -> 175.4 mm
- net BTN_BLUE: track 227.8 -> 223.7 mm
- net TFT SCL: track 93.5 -> 90.5 mm
- net TFT_LED: track 100.7 -> 99.2 mm
- net VRX: track 49.0 -> 50.0 mm
- net TFT_CS: track 84.8 -> 84.2 mm

Commit message: Fixed bugs need to be adressed
In this update, you know whats up.
Parts:
- added BZ1: Buzzer, Buzzer_Beeper:Buzzer_12x9.5RM7.6, B.Cu at (93.0, 57.5)
- J1: footprint Connector_PinSocket_2.54mm:PinSocket_1x09_P2.54mm_Vertical -> Connector_PinHeader_2.54mm:PinHeader_1x11_P2.54mm_Vertical; moved to F.Cu
- moved J1 6.02 mm to (108.5, 60.5), turned to 0 degrees
Connections:
- J1 pad 1: TFT_CS -> +3V3
- J1 pad 2: TFT_RST -> GND
- J1 pad 3: TFT_DC -> TFT_CS
- J1 pad 4: TFT_MOSI -> TFT_RST
- J1 pad 5: TFT_SCK -> TFT_DC
- J1 pad 6: TFT_LED -> TFT_MOSI
- J1 pad 7: TFT MISO -> TFT_SCK
- J1 pad 8: TFT SCL -> TFT_LED
- J1 pad 9: TFT SDA -> TFT MISO
Routing:
- net BUZZER: track 0.00 -> 140.5 mm
- net +3V3: track 199.2 -> 237.5 mm
- net TFT_MOSI: track 385.8 -> 402.8 mm, vias 0 -> 1
- net TFT_DC: track 94.5 -> 108.3 mm
- net TFT SCL: track 90.5 -> 99.4 mm
- net TFT_RST: track 141.8 -> 132.9 mm
- net SD_CS: track 175.4 -> 180.8 mm
- net TFT_CS: track 84.2 -> 85.2 mm
- net TFT_SCK: track 110.7 -> 111.6 mm
